Commit message: added, start and end state for test purpose (moveit collision problem)

File: config/panda_arm.xacro (robot description, xacro)
@@ -11,4 +11,22 @@
     </group>
     <!--GROUP STATES: Purpose: Define a named state for a particular group, in terms of joint values. This is useful to define states like 'folded arms'-->
+    <group_state name="start" group="panda_arm">
+      <joint name="panda_joint1" value="0.1557" />
+      <joint name="panda_joint2" value="-0.0492" />
+      <joint name="panda_joint3" value="0.0783" />
+      <joint name="panda_joint4" value="-1.4760" />
+      <joint name="panda_joint5" value="-1.08" />
+      <joint name="panda_joint6" value="2.853" />
+      <joint name="panda_joint7" value="1.841" />
+    </group_state>
+    <group_state name="end" group="panda_arm">
+      <joint name="panda_joint1" value="0.12392" />
+      <joint name="panda_joint2" value="1.2971" />
+      <joint name="panda_joint3" value="-2.582" />
+      <joint name="panda_joint4" value="-1.122" />
+      <joint name="panda_joint5" value="2.8679" />
+      <joint name="panda_joint6" value="1.858" />
+      <joint name="panda_joint7" value="0.28939" />
+    </group_state>
     <group_state name="ready" group="panda_arm">
       <joint name="panda_joint1" value="0" />
